Commit message: Editing hte files..

File: ros2_ws/src/hexapod_description/urdf/gazebo.xacro (robot description, xacro)
@@ -150,43 +150,24 @@
     <gazebo reference="lidar_link">
         <sensor name="laser" type="gpu_lidar">
-            <pose> 0 0 0 0 0 0 </pose>
+            <pose>0 0 0 0 0 0</pose>
             <always_on>true</always_on>
             <visualize>true</visualize>
             <update_rate>30</update_rate>
-            <topic>scan</topic>
-            <gz_frame_id>lidar_link</gz_frame_id>
+            <topic>/scan</topic>
             <lidar>
-            <scan>
-                <horizontal>
-                <samples>360</samples>
-                <min_angle>-3.14</min_angle>
-                <max_angle>3.14</max_angle>
-                </horizontal>
-            </scan>
-            <range>
-                <min>0.3</min>
-                <max>12</max>
-            </range>
+                <scan>
+                    <horizontal>
+                        <samples>360</samples>
+                        <resolution>1</resolution>
+                        <min_angle>-3.14159265359</min_angle>
+                        <max_angle>3.14159265359</max_angle>
+                    </horizontal>
+                </scan>
+                <range>
+                    <min>0.30</min>
+                    <max>12.0</max>
+                    <resolution>0.01</resolution>
+                </range>
             </lidar>
-        </sensor>
-    </gazebo>
-    <gazebo reference="base_link">
-        <sensor name="camera" type="camera">
-            <pose>0 0 0 0 0 0</pose>
-            <topic>camera/image_raw</topic>
-            <update_rate>30</update_rate>
-            <gz_frame_id>camera_link</gz_frame_id>
-            <camera>
-                <horizontal_fov>1.047</horizontal_fov> <image>
-                    <width>640</width>
-                    <height>480</height>
-                    <format>R8G8B8</format>
-                </image>
-                <clip>
-                    <near>0.1</near>
-                    <far>100</far>
-                </clip>
-            </camera>
-            <visualize>true</visualize>
         </sensor>
     </gazebo>

File: ros2_ws/src/hexapod_description/urdf/hexapod.urdf (robot description, URDF)
Before this commit: robot hexapod, 21 links, 20 joints
Links:
- removed link lidar_link-v1
- added link lidar_link, mass 0.5012486294496955; collision mesh filename=package://hexapod_description/meshes/lidar_link.stl scale=0.001 0.001 0.001; visual mesh filename=package://hexapod_description/meshes/lidar_link.stl scale=0.001 0.001 0.001
- link L1_Crus: mass 0.19082862947867688 -> 0.19082842966424732; geometry collision mesh filename=package://hexapod_description/meshes/L1_Crus.stl scale=0.001 0.001 0.001; visual mesh filename=package://hexapod_description/meshes/L1_Crus.stl scale=0.001 0.001 0.001
- link L1_Foot: geometry collision mesh filename=package://hexapod_description/meshes/L1_Foot.stl scale=0.001 0.001 0.001; visual mesh filename=package://hexapod_description/meshes/L1_Foot.stl scale=0.001 0.001 0.001
- link L1_Hip: geometry collision mesh filename=package://hexapod_description/meshes/L1_Hip.stl scale=0.001 0.001 0.001; visual mesh filename=package://hexapod_description/meshes/L1_Hip.stl scale=0.001 0.001 0.001
- link L2_Crus: mass 0.19082862947867688 -> 0.19082842966424732; geometry collision mesh filename=package://hexapod_description/meshes/L2_Crus.stl scale=0.001 0.001 0.001; visual mesh filename=package://hexapod_description/meshes/L2_Crus.stl scale=0.001 0.001 0.001
- link L2_Foot: geometry collision mesh filename=package://hexapod_description/meshes/L2_Foot.stl scale=0.001 0.001 0.001; visual mesh filename=package://hexapod_description/meshes/L2_Foot.stl scale=0.001 0.001 0.001
- link L2_Hip: geometry collision mesh filename=package://hexapod_description/meshes/L2_Hip.stl scale=0.001 0.001 0.001; visual mesh filename=package://hexapod_description/meshes/L2_Hip.stl scale=0.001 0.001 0.001
- link L3_Crus: mass 0.19082862947867688 -> 0.19082842966424732; geometry collision mesh filename=package://hexapod_description/meshes/L3_Crus.stl scale=0.001 0.001 0.001; visual mesh filename=package://hexapod_description/meshes/L3_Crus.stl scale=0.001 0.001 0.001
- link L3_Foot: geometry collision mesh filename=package://hexapod_description/meshes/L3_Foot.stl scale=0.001 0.001 0.001; visual mesh filename=package://hexapod_description/meshes/L3_Foot.stl scale=0.001 0.001 0.001
- link L3_Hip: geometry collision mesh filename=package://hexapod_description/meshes/L3_Hip.stl scale=0.001 0.001 0.001; visual mesh filename=package://hexapod_description/meshes/L3_Hip.stl scale=0.001 0.001 0.001
- link R1_Crus: mass 0.19082862947867688 -> 0.19082842966424732; geometry collision mesh filename=package://hexapod_description/meshes/R1_Crus.stl scale=0.001 0.001 0.001; visual mesh filename=package://hexapod_description/meshes/R1_Crus.stl scale=0.001 0.001 0.001
- link R1_Foot: geometry collision mesh filename=package://hexapod_description/meshes/R1_Foot.stl scale=0.001 0.001 0.001; visual mesh filename=package://hexapod_description/meshes/R1_Foot.stl scale=0.001 0.001 0.001
- link R1_Hip: geometry collision mesh filename=package://hexapod_description/meshes/R1_Hip.stl scale=0.001 0.001 0.001; visual mesh filename=package://hexapod_description/meshes/R1_Hip.stl scale=0.001 0.001 0.001
- link R2_Crus: mass 0.19082862947867688 -> 0.19082842966424732; geometry collision mesh filename=package://hexapod_description/meshes/R2_Crus.stl scale=0.001 0.001 0.001; visual mesh filename=package://hexapod_description/meshes/R2_Crus.stl scale=0.001 0.001 0.001
- link R2_Foot: geometry collision mesh filename=package://hexapod_description/meshes/R2_Foot.stl scale=0.001 0.001 0.001; visual mesh filename=package://hexapod_description/meshes/R2_Foot.stl scale=0.001 0.001 0.001
- link R2_Hip: geometry collision mesh filename=package://hexapod_description/meshes/R2_Hip.stl scale=0.001 0.001 0.001; visual mesh filename=package://hexapod_description/meshes/R2_Hip.stl scale=0.001 0.001 0.001
- link R3_Crus: mass 0.19082862947867688 -> 0.19082842966424732; geometry collision mesh filename=package://hexapod_description/meshes/R3_Crus.stl scale=0.001 0.001 0.001; visual mesh filename=package://hexapod_description/meshes/R3_Crus.stl scale=0.001 0.001 0.001
- link R3_Foot: geometry collision mesh filename=package://hexapod_description/meshes/R3_Foot.stl scale=0.001 0.001 0.001; visual mesh filename=package://hexapod_description/meshes/R3_Foot.stl scale=0.001 0.001 0.001
- link R3_Hip: geometry collision mesh filename=package://hexapod_description/meshes/R3_Hip.stl scale=0.001 0.001 0.001; visual mesh filename=package://hexapod_description/meshes/R3_Hip.stl scale=0.001 0.001 0.001
- link base_link: mass 10.813766886555406 -> 1.813766886555406; geometry collision mesh filename=package://hexapod_description/meshes/base_link.stl scale=0.001 0.001 0.001; visual mesh filename=package://hexapod_description/meshes/base_link.stl scale=0.001 0.001 0.001
Joints:
- joint L1_Ankle_Joint: axis -1.0 7.59658234058801e-46 4.718652233545131e-15 -> 0.0 1.0 -7.480279667283062e-17; origin xyz=8.881784197001253e-17 2.6645352591003756e-17 -0.07000000000000003 rpy=-1.5707963267948961 1.7627500921248386e-32 8.043744362719904e-31 -> xyz=0.07000000000000003 0.0 0.0 rpy=-1.5707963267948961 5.1796479912722884e-61 -1.3063417489326808e-45; type revolute -> continuous
- joint L1_Hip_Joint: origin xyz=0.13403352999999998 -0.003461909999999868 0.07190117 rpy=6.008386403513597e-16 6.9388939039072014e-18 -1.5707963267948961 -> xyz=0.13403352999999996 -0.003461909999999939 0.07190117 rpy=6.285942159669887e-16 -0.0 0.0; type revolute -> continuous
- joint L1_Knee_Joint: axis 1.0 -5.3637286999234275e-62 1.1622299354398722e-15 -> 0.0 -3.9650022633849155e-16 1.0; origin xyz=0.03361222999999997 0.03989999999999997 -0.033725000000000026 rpy=1.5707963267948957 -1.3138613440828752e-47 -2.090158182670701e-32 -> xyz=0.03989999999999997 -0.03361223000000004 -0.03372499999999998 rpy=1.5707963267948957 -0.0 0.0; type revolute -> continuous
- joint L2_Ankle_Joint: axis -1.0 1.8212480051892797e-60 4.7186522335451305e-15 -> 0.0 1.0 -7.480279667283062e-17; origin xyz=-2.708944180085382e-16 -5.329070518200751e-17 -0.07 rpy=-1.5707963267948972 1.9409610039179162e-32 4.7832386332694783e-32 -> xyz=0.07000000000000002 0.0 0.0 rpy=-1.5707963267948972 -1.9039111407057832e-59 -2.640308508991052e-44; type revolute -> continuous
- joint L2_Hip_Joint: origin xyz=0.1552999999999999 0.09500000000000006 0.0712 rpy=6.47653695138311e-16 6.9388939039072014e-18 -1.5707963267948961 -> xyz=0.15529999999999994 0.09500000000000006 0.0712 rpy=6.7540927075394e-16 -0.0 0.0; type revolute -> continuous
- joint L2_Knee_Joint: axis 1.0 -7.392375377700111e-47 -3.8498572664985686e-15 -> -0.0 7.2109419570568655e-16 1.0; origin xyz=0.033612220000000005 0.03989999999999997 -0.033725000000000026 rpy=1.5707963267948966 -1.3239509656106505e-47 -1.9602203033617853e-32 -> xyz=0.039900000000000005 -0.033612220000000026 -0.03372499999999998 rpy=1.5707963267948966 -0.0 0.0; type revolute -> continuous
- joint L3_Ankle_Joint: axis -1.0 1.1801800379278693e-46 4.718652233545132e-15 -> 0.0 1.0 -7.480279667283062e-17; origin xyz=-3.2862601528904633e-16 -5.773159728050814e-17 -0.07 rpy=-1.5707963267948974 2.3859822435111286e-32 1.6247875503541474e-30 -> xyz=0.06999999999999998 0.0 0.0 rpy=-1.5707963267948974 -2.4135408364719946e-59 -2.826793622035183e-44; type revolute -> continuous
- joint L3_Hip_Joint: origin xyz=0.13403341999999988 0.19346199999999997 0.0709 rpy=4.873178960340447e-16 6.9388939039072014e-18 -1.5707963267948961 -> xyz=0.13403341999999996 0.19346200000000002 0.0709 rpy=5.150734716496737e-16 -0.0 0.0; type revolute -> continuous
- joint L3_Knee_Joint: axis 1.0 2.0200727857016129e-47 -4.776934255052703e-15 -> -0.0 8.538086465379591e-16 1.0; origin xyz=0.033612230000000014 0.039899999999999984 -0.033725000000000026 rpy=1.570796326794897 -1.2388761116857788e-47 -2.4052415429548625e-32 -> xyz=0.03990000000000002 -0.033612230000000014 -0.033724999999999984 rpy=1.570796326794897 -0.0 0.0; type revolute -> continuous
- joint Lidar_Joint: child lidar_link-v1 -> lidar_link
- joint R1_Ankle_Joint: axis 0.999776 0.021186 -4.722648697290969e-15 -> -0.0 -1.0 7.480279667283062e-17; origin xyz=0.0014829900000003261 7.105427357601002e-17 0.06998429000000002 rpy=-1.5707963267948974 -3.4694469519504815e-18 3.4694469519480348e-18 -> xyz=-0.07000000000000002 0.0 0.0 rpy=-1.5707963267948974 -8.694335908329952e-33 -4.894512470596831e-34; type revolute -> continuous
- joint R1_Hip_Joint: origin xyz=-0.003944869999999936 -0.0033736899999999535 0.07150000000000001 rpy=-6.435241798119282e-16 6.9388939039072014e-18 -1.5707963267948961 -> xyz=-0.003944870000000052 -0.0033736899999999535 0.07150000000000001 rpy=-6.157686041962991e-16 -0.0 0.0; type revolute -> continuous
- joint R1_Knee_Joint: axis -0.999776 2.1429753129425157e-17 0.021186000000004618 -> 8.694335908329952e-33 -1.0115053870209175e-15 -1.0; origin xyz=-0.03275938000000005 -0.040603139999999975 -0.033725000000000026 rpy=1.5707963267948983 3.9229407610357025e-31 3.4694469519504846e-18 -> xyz=-0.03990000000000004 0.03361222000000002 -0.033724999999999984 rpy=1.5707963267948983 -5.3536990866860975e-48 8.694335908329952e-33; type revolute -> continuous
- joint R2_Ankle_Joint: axis 1.0 -2.1771648783370645e-47 -4.7186522335451305e-15 -> 0.0 -1.0 7.480279667283062e-17; origin xyz=1.1990408665951691e-16 6.661338147750939e-17 0.07 rpy=-1.5707963267948974 -9.269768496042548e-32 5.825108194838518e-31 -> xyz=-0.07000000000000002 0.0 0.0 rpy=-1.5707963267948974 -3.481608803689402e-33 1.0186570131224499e-31; type revolute -> continuous
- joint R2_Hip_Joint: origin xyz=-0.02529999999999997 0.09499999999999999 0.0712 rpy=-8.903513958032982e-16 6.9388939039072014e-18 -1.5707963267948961 -> xyz=-0.025300000000000048 0.09500000000000006 0.0712 rpy=-8.625958201876691e-16 -0.0 0.0; type revolute -> continuous
- joint R2_Knee_Joint: axis -1.0 -2.0680855234740677e-47 1.7116111111633693e-15 -> 3.4816088036894984e-33 -9.473014393433699e-16 -1.0; origin xyz=-0.033612220000000005 -0.039899999999999984 -0.03372500000000003 rpy=1.5707963267948983 2.4651903288156496e-32 1.4180889854230056e-31 -> xyz=-0.039900000000000005 0.03361222000000003 -0.03372499999999997 rpy=1.5707963267948983 -3.0032212015911526e-48 3.4816088036894984e-33; type revolute -> continuous
- joint R3_Ankle_Joint: axis 1.0 9.86076131526266e-32 -4.718652233545129e-15 -> 0.0 -1.0 7.480279667283062e-17; origin xyz=-2.486899575160351e-16 4.884981308350689e-17 0.06999999999999998 rpy=-1.5707963267948972 -1.1559672828576987e-31 -1.320472174686651e-30 -> xyz=-0.07000000000000002 0.0 0.0 rpy=-1.5707963267948972 -8.502863783488482e-34 3.021914200080796e-31; type revolute -> continuous
- joint R3_Hip_Joint: origin xyz=-0.00403342000000003 0.19346199999999988 0.0709 rpy=-6.230017662244101e-16 6.9388939039072014e-18 -1.5707963267948961 -> xyz=-0.004033420000000057 0.19346200000000002 0.0709 rpy=-5.952461906087811e-16 -0.0 0.0; type revolute -> continuous
- joint R3_Knee_Joint: axis -1.0 -9.86076131526265e-32 -3.58465812034788e-15 -> 8.502863783490581e-34 -6.944343755255036e-16 -1.0; origin xyz=-0.03361221999999998 -0.03989999999999998 -0.033725000000000026 rpy=1.570796326794898 -9.860761315262654e-32 1.1540413529133016e-31 -> xyz=-0.03989999999999999 0.03361222000000002 -0.033724999999999984 rpy=1.570796326794898 -5.061297276388136e-49 8.502863783490581e-34; type revolute -> continuous
- joint base_joint: origin xyz=0.0 0.0 0.0 rpy=0.0 0.0 0.0 -> xyz=0.0 0.0 0.05 rpy=0.0 0.0 0.0

File: ros2_ws/src/hexapod_description/urdf/hexapod.xacro (robot description, xacro)
@@ -433,5 +433,5 @@
             <origin xyz="-0.035950900915733504 -0.01809786515993314 -0.03369999999999962" rpy="-1.570796326794898 9.568681466994664e-17 0.5497787143782145" />
             <geometry>
-                <mesh filename="meshes/lidar_link.stl" scale="0.001 0.001 0.001" />
+                <mesh filename="package://hexapod_description/meshes/lidar_link.stl" scale="0.001 0.001 0.001" />
             </geometry>
             <material name="Red">
@@ -442,5 +442,5 @@
             <origin xyz="-0.035950900915733504 -0.01809786515993314 -0.03369999999999962" rpy="-1.570796326794898 9.568681466994664e-17 0.5497787143782145" />
             <geometry>
-                <mesh filename="meshes/lidar_link.stl" scale="0.001 0.001 0.001" />
+                <mesh filename="package://hexapod_description/meshes/lidar_link.stl" scale="0.001 0.001 0.001" />
             </geometry>
         </collision>
@@ -560,5 +560,5 @@
         <axis xyz="0.0 -1.0 7.480279667283062e-17" />
     </joint>
-    <joint name="base_link_Lidar_Joint" type="fixed">
+    <joint name="Lidar_Joint" type="fixed">
         <origin xyz="0.046999999999999986 0.09400000000000003 0.150669" rpy="3.141592653589793 6.9388939039072014e-18 -1.5707963267948961" />
         <parent link="base_link" />
