Commit message: Changed the collision to mesh collision

File: ros2_ws/src/hexapod_description/urdf/hexapod.xacro (robot description, xacro)
@@ -14,5 +14,5 @@
             </geometry>
             <material name="Black">
-                <color rgba="0.000000 0.000000 0.000000 1.000000"/>
+                <color rgba="0.0250000 0.02500000 0.02500000 1.00000"/>
             </material>
         </visual>
@@ -20,5 +20,5 @@
             <origin xyz="0.0 0.0 0.0" rpy="0.0 0.0 0.0" />
             <geometry>
-                <box size="0.34 0.25 0.10" />
+                <mesh filename="package://hexapod_description/meshes/base_link.stl" scale="0.001 0.001 0.001" />
             </geometry>
         </collision>
@@ -42,5 +42,5 @@
             <origin xyz="-7.947591029733303e-11 2.8394247545868725e-05 -0.03750000103512392" rpy="3.9470377442356937e-16 -0.0 0.0" />
             <geometry>
-                <box size="0.09 0.09 0.08" />
+                <mesh filename="package://hexapod_description/meshes/L1_Hip.stl" scale="0.001 0.001 0.001" />
             </geometry>
         </collision>
@@ -64,5 +64,5 @@
             <origin xyz="2.3092638912203257e-16 2.8396418664446987e-05 -0.037500000000000304" rpy="3.947037744235681e-16 7.394140421080006e-63 1.0947644252537633e-47" />
             <geometry>
-                <box size="0.09 0.09 0.08" />
+                <mesh filename="package://hexapod_description/meshes/L2_Hip.stl" scale="0.001 0.001 0.001" />
             </geometry>
         </collision>
@@ -86,5 +86,5 @@
             <origin xyz="-1.8717173055904367e-09 2.8395102015679187e-05 -0.03749999999999909" rpy="3.947037744235681e-16 -0.0 0.0" />
             <geometry>
-                <box size="0.09 0.09 0.08" />
+                <mesh filename="package://hexapod_description/meshes/L3_Hip.stl" scale="0.001 0.001 0.001" />
             </geometry>
         </collision>
@@ -108,5 +108,5 @@
             <origin xyz="-5.436926464597036e-10 -2.8396543466868707e-05 -0.0375000000000004" rpy="3.94703774423568e-16 2.4310372503823276e-15 3.141592653589793" />
             <geometry>
-                <box size="0.09 0.09 0.08" />
+                <mesh filename="package://hexapod_description/meshes/R1_Hip.stl" scale="0.001 0.001 0.001" />
             </geometry>
         </collision>
@@ -130,5 +130,5 @@
             <origin xyz="5.329070518200751e-17 -2.839641866355881e-05 -0.03749999999999999" rpy="3.94703774423568e-16 9.526600354478707e-17 3.141592653589793" />
             <geometry>
-                <box size="0.09 0.09 0.08" />
+                <mesh filename="package://hexapod_description/meshes/R2_Hip.stl" scale="0.001 0.001 0.001" />
             </geometry>
         </collision>
@@ -152,5 +152,5 @@
             <origin xyz="1.8717173855264947e-09 -2.839773531169598e-05 -0.0374999999999994" rpy="3.947037744235682e-16 -8.475327317661527e-16 3.141592653589793" />
             <geometry>
-                <box size="0.09 0.09 0.08" />
+                <mesh filename="package://hexapod_description/meshes/R3_Hip.stl" scale="0.001 0.001 0.001" />
             </geometry>
         </collision>
@@ -174,5 +174,5 @@
             <origin xyz="-0.018685768413435184 0.017921808755716372 -0.011675028544473465" rpy="2.9586803559888716e-15 9.464173730837164e-15 -3.141592653589791" />
             <geometry>
-                <box size="0.15 0.06 0.06" />
+                <mesh filename="package://hexapod_description/meshes/R1_Crus.stl" scale="0.001 0.001 0.001" />
             </geometry>
         </collision>
@@ -196,5 +196,5 @@
             <origin xyz="-0.05131423213025757 -0.017921808755717222 -0.01167502866927641" rpy="-3.2267052699708074e-15 2.8845764424670263e-15 2.177306834595132e-16" />
             <geometry>
-                <box size="0.15 0.06 0.06" />
+                <mesh filename="package://hexapod_description/meshes/R2_Crus.stl" scale="0.001 0.001 0.001" />
             </geometry>
         </collision>
@@ -218,5 +218,5 @@
             <origin xyz="-0.0513142302585405 -0.017921808755716497 -0.011675027352628008" rpy="-2.453621512756187e-15 8.180845673978275e-15 -7.250680518514371e-16" />
             <geometry>
-                <box size="0.15 0.06 0.06" />
+                <mesh filename="package://hexapod_description/meshes/R3_Crus.stl" scale="0.001 0.001 0.001" />
             </geometry>
         </collision>
@@ -240,5 +240,5 @@
             <origin xyz="0.018685767790268776 0.017921807720593708 0.011675020840395725" rpy="-3.1415926535897922 -3.556422298105262e-15 -3.77670496181703e-30" />
             <geometry>
-                <box size="0.15 0.06 0.06" />
+                <mesh filename="package://hexapod_description/meshes/L1_Crus.stl" scale="0.001 0.001 0.001" />
             </geometry>
         </collision>
@@ -262,5 +262,5 @@
             <origin xyz="0.018685767869742236 0.017921808755716546 0.011675028669276171" rpy="-3.1415926535897922 -8.5685095000437e-15 -9.204085185479184e-30" />
             <geometry>
-                <box size="0.15 0.06 0.06" />
+                <mesh filename="package://hexapod_description/meshes/L2_Crus.stl" scale="0.001 0.001 0.001" />
             </geometry>
         </collision>
@@ -284,5 +284,5 @@
             <origin xyz="0.018685765998024823 0.017921808755717642 0.011675019985925648" rpy="-3.1415926535897922 -9.495586488597836e-15 -8.631228484744494e-30" />
             <geometry>
-                <box size="0.15 0.06 0.06" />
+                <mesh filename="package://hexapod_description/meshes/L3_Crus.stl" scale="0.001 0.001 0.001" />
             </geometry>
         </collision>
@@ -306,5 +306,5 @@
             <origin xyz="-0.01010000007948257 0.019400003427672525 -0.02056704031521055" rpy="6.610591211137782e-14 9.860761315262522e-32 -7.376125237048963e-48" />
             <geometry>
-                <box size="0.18 0.07 0.025" />
+                <mesh filename="package://hexapod_description/meshes/L1_Foot.stl" scale="0.001 0.001 0.001" />
             </geometry>
         </collision>
@@ -328,5 +328,5 @@
             <origin xyz="-0.010100000000000726 0.019399995598791568 -0.02056703928008564" rpy="3.921169725428927e-14 3.697785493220852e-32 -2.766046963891421e-48" />
             <geometry>
-                <box size="0.18 0.07 0.025" />
+                <mesh filename="package://hexapod_description/meshes/L2_Foot.stl" scale="0.001 0.001 0.001" />
             </geometry>
         </collision>
@@ -350,5 +350,5 @@
             <origin xyz="-0.010100001871717198 0.019400004282141385 -0.020567039280084735" rpy="-1.0782612974161142e-15 -2.826793622035183e-44 2.114520685451522e-60" />
             <geometry>
-                <box size="0.18 0.07 0.025" />
+                <mesh filename="package://hexapod_description/meshes/L3_Foot.stl" scale="0.001 0.001 0.001" />
             </geometry>
         </collision>
@@ -372,5 +372,5 @@
             <origin xyz="0.010099999456307032 -0.019399995723592314 -0.020567039280086543" rpy="-3.744677003792175e-15 2.4310372503823272e-15 -3.141592653589793" />
             <geometry>
-                <box size="0.18 0.07 0.025" />
+                <mesh filename="package://hexapod_description/meshes/R1_Foot.stl" scale="0.001 0.001 0.001" />
             </geometry>
         </collision>
@@ -394,5 +394,5 @@
             <origin xyz="0.010099999999999625 -0.019399995598789698 -0.020567039280085676" rpy="2.824311711540962e-16 9.526600354478716e-17 3.141592653589793" />
             <geometry>
-                <box size="0.18 0.07 0.025" />
+                <mesh filename="package://hexapod_description/meshes/R2_Foot.stl" scale="0.001 0.001 0.001" />
             </geometry>
         </collision>
@@ -416,5 +416,5 @@
             <origin xyz="0.010100001871717269 -0.019399996915439015 -0.020567039280085346" rpy="-2.089940004168009e-16 -8.475327317661533e-16 3.141592653589793" />
             <geometry>
-                <box size="0.18 0.07 0.025" />
+                <mesh filename="package://hexapod_description/meshes/R3_Foot.stl" scale="0.001 0.001 0.001" />
             </geometry>
         </collision>

Commit message: The Hexapod is now standing properly

File: ros2_ws/src/hexapod_description/urdf/hexapod.xacro (robot description, xacro)
@@ -5,5 +5,5 @@
         <inertial>
             <origin xyz="0.06531354373116458 0.09547813117381193 0.055845566802461395" rpy="0.0 0.0 0.0" />
-            <mass value="10.813766886555406" />
+            <mass value="1.813766886555406" />
             <inertia ixx="0.052834066282912866" iyy="0.038235219700231526" izz="0.058132624055021655" ixy="-6.396865406510826e-05" iyz="-0.001076769870526382" ixz="-8.416476796523591e-05" />
         </inertial>
@@ -422,5 +422,5 @@
     <joint name="base_joint" type="fixed">
         <!-- base_footprint is the ground reference. Raise the body so the leg feet can reach z=0. -->
-        <origin xyz="0.0 0.0 0.1446" rpy="0.0 0.0 0.0" />
+        <origin xyz="0.0 0.0 0.05" rpy="0.0 0.0 0.0" />
         <parent link="base_footprint" />
         <child link="base_link" />

Commit message: Seperated Files...

File: ros2_ws/src/hexapod_description/urdf/hexapod.xacro (robot description, xacro)
@@ -1,4 +1,8 @@
 <?xml version='1.0' encoding='utf-8'?>
-<robot name="hexapod">
+<robot name="hexapod" xmlns:xacro="http://www.ros.org/wiki/xacro">
+  <!-- Include materials -->
+  <xacro:include filename="$(find hexapod_description)/urdf/materials.xacro"/>
+  <!-- Include gazebo -->
+  <xacro:include filename="$(find hexapod_description)/urdf/gazebo.xacro"/>
     <link name="base_footprint"/>
     <link name="base_link">
@@ -417,4 +421,26 @@
             <geometry>
                 <mesh filename="package://hexapod_description/meshes/R3_Foot.stl" scale="0.001 0.001 0.001" />
+            </geometry>
+        </collision>
+    </link>
+    <link name="lidar_link">
+        <inertial>
+            <origin xyz="-0.027461976774698915 -0.018137996208371785 -0.01992249948325206" rpy="0.0 -0.0 0.0" />
+            <mass value="0.5012486294496955" />
+            <inertia ixx="0.00016602133606471135" iyy="0.00032461555354666195" izz="0.0003217777330464164" ixy="-8.489893768956169e-07" iyz="-1.2052271770585847e-06" ixz="-8.741763903184424e-06" />
+        </inertial>
+        <visual name="lidar_link_visual">
+            <origin xyz="-0.035950900915733504 -0.01809786515993314 -0.03369999999999962" rpy="-1.570796326794898 9.568681466994664e-17 0.5497787143782145" />
+            <geometry>
+                <mesh filename="meshes/lidar_link.stl" scale="0.001 0.001 0.001" />
+            </geometry>
+            <material name="Red">
+                <color rgba="1.000000 0.000000 0.000000 1.000000"/>
+            </material>
+        </visual>
+        <collision name="lidar_link_collision">
+            <origin xyz="-0.035950900915733504 -0.01809786515993314 -0.03369999999999962" rpy="-1.570796326794898 9.568681466994664e-17 0.5497787143782145" />
+            <geometry>
+                <mesh filename="meshes/lidar_link.stl" scale="0.001 0.001 0.001" />
             </geometry>
         </collision>
@@ -534,148 +560,8 @@
         <axis xyz="0.0 -1.0 7.480279667283062e-17" />
     </joint>
-  <!-- Simplified primitive collision geometry is used because DART cannot
-       construct the CAD STL collision meshes reliably.  Keep STL as visual only. -->
-  <gazebo reference="base_link">
-    <mu1>0.6</mu1>
-    <mu2>0.6</mu2>
-  </gazebo>
-  <gazebo reference="L1_Foot">
-    <mu1>1.0</mu1>
-    <mu2>1.0</mu2>
-    <kp>100000.0</kp>
-    <kd>10.0</kd>
-  </gazebo>
-  <gazebo reference="L2_Foot">
-    <mu1>1.0</mu1>
-    <mu2>1.0</mu2>
-    <kp>100000.0</kp>
-    <kd>10.0</kd>
-  </gazebo>
-  <gazebo reference="L3_Foot">
-    <mu1>1.0</mu1>
-    <mu2>1.0</mu2>
-    <kp>100000.0</kp>
-    <kd>10.0</kd>
-  </gazebo>
-  <gazebo reference="R1_Foot">
-    <mu1>1.0</mu1>
-    <mu2>1.0</mu2>
-    <kp>100000.0</kp>
-    <kd>10.0</kd>
-  </gazebo>
-  <gazebo reference="R2_Foot">
-    <mu1>1.0</mu1>
-    <mu2>1.0</mu2>
-    <kp>100000.0</kp>
-    <kd>10.0</kd>
-  </gazebo>
-  <gazebo reference="R3_Foot">
-    <mu1>1.0</mu1>
-    <mu2>1.0</mu2>
-    <kp>100000.0</kp>
-    <kd>10.0</kd>
-  </gazebo>
-  <!-- ROS 2 Control interface for Gazebo Harmonic / gz_ros2_control. -->
-  <ros2_control name="GazeboSimSystem" type="system">
-    <hardware>
-      <plugin>gz_ros2_control/GazeboSimSystem</plugin>
-    </hardware>
-    <joint name="L1_Hip_Joint">
-      <command_interface name="position"/>
-      <state_interface name="position"/>
-      <state_interface name="velocity"/>
-    </joint>
-    <joint name="L2_Hip_Joint">
-      <command_interface name="position"/>
-      <state_interface name="position"/>
-      <state_interface name="velocity"/>
-    </joint>
-    <joint name="L3_Hip_Joint">
-      <command_interface name="position"/>
-      <state_interface name="position"/>
-      <state_interface name="velocity"/>
-    </joint>
-    <joint name="R1_Hip_Joint">
-      <command_interface name="position"/>
-      <state_interface name="position"/>
-      <state_interface name="velocity"/>
-    </joint>
-    <joint name="R2_Hip_Joint">
-      <command_interface name="position"/>
-      <state_interface name="position"/>
-      <state_interface name="velocity"/>
-    </joint>
-    <joint name="R3_Hip_Joint">
-      <command_interface name="position"/>
-      <state_interface name="position"/>
-      <state_interface name="velocity"/>
-    </joint>
-    <joint name="R1_Knee_Joint">
-      <command_interface name="position"/>
-      <state_interface name="position"/>
-      <state_interface name="velocity"/>
-    </joint>
-    <joint name="R2_Knee_Joint">
-      <command_interface name="position"/>
-      <state_interface name="position"/>
-      <state_interface name="velocity"/>
-    </joint>
-    <joint name="R3_Knee_Joint">
-      <command_interface name="position"/>
-      <state_interface name="position"/>
-      <state_interface name="velocity"/>
-    </joint>
-    <joint name="L1_Knee_Joint">
-      <command_interface name="position"/>
-      <state_interface name="position"/>
-      <state_interface name="velocity"/>
-    </joint>
-    <joint name="L2_Knee_Joint">
-      <command_interface name="position"/>
-      <state_interface name="position"/>
-      <state_interface name="velocity"/>
-    </joint>
-    <joint name="L3_Knee_Joint">
-      <command_interface name="position"/>
-      <state_interface name="position"/>
-      <state_interface name="velocity"/>
-    </joint>
-    <joint name="L1_Ankle_Joint">
-      <command_interface name="position"/>
-      <state_interface name="position"/>
-      <state_interface name="velocity"/>
-    </joint>
-    <joint name="L2_Ankle_Joint">
-      <command_interface name="position"/>
-      <state_interface name="position"/>
-      <state_interface name="velocity"/>
-    </joint>
-    <joint name="L3_Ankle_Joint">
-      <command_interface name="position"/>
-      <state_interface name="position"/>
-      <state_interface name="velocity"/>
-    </joint>
-    <joint name="R1_Ankle_Joint">
-      <command_interface name="position"/>
-      <state_interface name="position"/>
-      <state_interface name="velocity"/>
-    </joint>
-    <joint name="R2_Ankle_Joint">
-      <command_interface name="position"/>
-      <state_interface name="position"/>
-      <state_interface name="velocity"/>
-    </joint>
-    <joint name="R3_Ankle_Joint">
-      <command_interface name="position"/>
-      <state_interface name="position"/>
-      <state_interface name="velocity"/>
-    </joint>
-  </ros2_control>
-  <gazebo>
-    <plugin filename="libgz_ros2_control-system.so"
-            name="gz_ros2_control::GazeboSimROS2ControlPlugin">
-      <parameters>$(find hexapod_controller)/config/controllers.yaml</parameters>
-      <controller_manager_name>controller_manager</controller_manager_name>
-    </plugin>
-  </gazebo>
+    <joint name="base_link_Lidar_Joint" type="fixed">
+        <origin xyz="0.046999999999999986 0.09400000000000003 0.150669" rpy="3.141592653589793 6.9388939039072014e-18 -1.5707963267948961" />
+        <parent link="base_link" />
+        <child link="lidar_link" />
+    </joint>
 </robot>
