Commit message: Updated RViz

File: ros2_ws/src/hexapod_description/urdf/hexapod.xacro (robot description, xacro)
@@ -8,7 +8,7 @@
     <link name="base_link">
         <inertial>
-            <origin xyz="0.06531354373116458 0.09547813117381193 0.055845566802461395" rpy="0.0 0.0 0.0" />
-            <mass value="1.813766886555406" />
-            <inertia ixx="0.052834066282912866" iyy="0.038235219700231526" izz="0.058132624055021655" ixy="-6.396865406510826e-05" iyz="-0.001076769870526382" ixz="-8.416476796523591e-05" />
+            <origin xyz="0.00031354372899712206 0.00047813117064395065 0.05584556680246142" rpy="0.0 0.0 0.0" />
+            <mass value="10.813766886555406" />
+            <inertia ixx="0.05283406628620018" iyy="0.03823521970176997" izz="0.0581326240598471" ixy="-6.396865631374618e-05" iyz="-0.0010767698724394807" ixz="-8.416476927420918e-05" />
         </inertial>
         <visual name="base_link_visual">
@@ -18,5 +18,5 @@
             </geometry>
             <material name="Black">
-                <color rgba="0.0250000 0.02500000 0.02500000 1.00000"/>
+                <color rgba="0.0 0.0 0.0 1.0"/>
             </material>
         </visual>
@@ -30,19 +30,22 @@
     <link name="L1_Hip">
         <inertial>
-            <origin xyz="0.036074048808862946 0.0008949127635549203 -0.027882387987432537" rpy="0.0 -0.0 0.0" />
+            <origin xyz="-0.0008949168650770112 0.03607405149828697 -0.02788238798743265" rpy="0.0 -0.0 0.0" />
             <mass value="0.6313074615876145" />
-            <inertia ixx="0.00032774839375865165" iyy="0.0003956699823553893" izz="0.0002593342441534908" ixy="-7.110380838515507e-06" iyz="1.8547901923319203e-05" ixz="1.1372181455404608e-05" />
+            <inertia ixx="0.00039566998235538754" iyy="0.0003277483937586577" izz="0.0002593342441534925" ixy="7.110380838514634e-06" iyz="1.1372181455403983e-05" ixz="-1.8547901923319647e-05" />
         </inertial>
         <visual name="L1_Hip_visual">
-            <origin xyz="-7.947591029733303e-11 2.8394247545868725e-05 -0.03750000103512392" rpy="3.9470377442356937e-16 -0.0 0.0" />
+            <origin xyz="-2.8398349067977334e-05 2.6099480443519953e-09 -0.03750000103512398" rpy="8.220700671772462e-16 1.7538274861003726e-15 1.5707963267948968" />
             <geometry>
                 <mesh filename="package://hexapod_description/meshes/L1_Hip.stl" scale="0.001 0.001 0.001" />
             </geometry>
             <material name="Red">
-                <color rgba="1.000000 0.000000 0.000000 1.000000"/>
+                <color rgba="1.0 0.0 0.0 1.0"/>
+            </material>
+            <material name="Red">
+                <color rgba="1.0 0.0 0.0 1.0"/>
             </material>
         </visual>
         <collision name="L1_Hip_collision">
-            <origin xyz="-7.947591029733303e-11 2.8394247545868725e-05 -0.03750000103512392" rpy="3.9470377442356937e-16 -0.0 0.0" />
+            <origin xyz="-2.8398349067977334e-05 2.6099480443519953e-09 -0.03750000103512398" rpy="8.220700671772462e-16 1.7538274861003726e-15 1.5707963267948968" />
             <geometry>
                 <mesh filename="package://hexapod_description/meshes/L1_Hip.stl" scale="0.001 0.001 0.001" />
@@ -52,19 +55,19 @@
     <link name="L2_Hip">
         <inertial>
-            <origin xyz="0.03607404944183094 0.0008949172145009408 -0.027882387844535943" rpy="0.0 -0.0 0.0" />
+            <origin xyz="-0.0008949213160230321 0.03607405213125471 -0.027882387844536016" rpy="0.0 -0.0 0.0" />
             <mass value="0.6313073388499962" />
-            <inertia ixx="0.0003277483586499371" iyy="0.00039566996489754855" izz="0.00025933422894452995" ixy="-7.110376138875333e-06" iyz="1.8547895317003865e-05" ixz="1.1372177166432535e-05" />
+            <inertia ixx="0.00039566996489754855" iyy="0.0003277483586499373" izz="0.0002593342289445282" ixy="7.110376138875355e-06" iyz="1.1372177166433766e-05" ixz="-1.8547895317004048e-05" />
         </inertial>
         <visual name="L2_Hip_visual">
-            <origin xyz="2.3092638912203257e-16 2.8396418664446987e-05 -0.037500000000000304" rpy="3.947037744235681e-16 7.394140421080006e-63 1.0947644252537633e-47" />
+            <origin xyz="-2.8400520186542823e-05 2.689423990176465e-09 -0.037500000000000276" rpy="1.1741964537361185e-15 2.4928608461965563e-15 1.5707963267948968" />
             <geometry>
                 <mesh filename="package://hexapod_description/meshes/L2_Hip.stl" scale="0.001 0.001 0.001" />
             </geometry>
             <material name="Red">
-                <color rgba="1.000000 0.000000 0.000000 1.000000"/>
+                <color rgba="1.0 0.0 0.0 1.0"/>
             </material>
         </visual>
         <collision name="L2_Hip_collision">
-            <origin xyz="2.3092638912203257e-16 2.8396418664446987e-05 -0.037500000000000304" rpy="3.947037744235681e-16 7.394140421080006e-63 1.0947644252537633e-47" />
+            <origin xyz="-2.8400520186542823e-05 2.689423990176465e-09 -0.037500000000000276" rpy="1.1741964537361185e-15 2.4928608461965563e-15 1.5707963267948968" />
             <geometry>
                 <mesh filename="package://hexapod_description/meshes/L2_Hip.stl" scale="0.001 0.001 0.001" />
@@ -74,19 +77,19 @@
     <link name="L3_Hip">
         <inertial>
-            <origin xyz="0.03607404682162757 0.0008949164118949327 -0.02788238784453293" rpy="0.0 -0.0 0.0" />
+            <origin xyz="-0.0008949205134169525 0.036074049511051455 -0.027882387844533032" rpy="0.0 -0.0 0.0" />
             <mass value="0.6313073388499971" />
-            <inertia ixx="0.00032774835013938027" iyy="0.0003956699570360784" izz="0.0002593342125795546" ixy="-7.110383350401172e-06" iyz="1.854789276545464e-05" ixz="1.1372179198901924e-05" />
+            <inertia ixx="0.00039566995703608013" iyy="0.00032774835013938027" izz="0.0002593342125795494" ixy="7.110383350402036e-06" iyz="1.1372179198903025e-05" ixz="-1.8547892765454083e-05" />
         </inertial>
         <visual name="L3_Hip_visual">
-            <origin xyz="-1.8717173055904367e-09 2.8395102015679187e-05 -0.03749999999999909" rpy="3.947037744235681e-16 -0.0 0.0" />
+            <origin xyz="-2.839920353769898e-05 8.17706542477481e-10 -0.0374999999999991" rpy="9.861050790162203e-16 2.814169320963183e-15 1.5707963267948968" />
             <geometry>
                 <mesh filename="package://hexapod_description/meshes/L3_Hip.stl" scale="0.001 0.001 0.001" />
             </geometry>
             <material name="Red">
-                <color rgba="1.000000 0.000000 0.000000 1.000000"/>
+                <color rgba="1.0 0.0 0.0 1.0"/>
             </material>
         </visual>
         <collision name="L3_Hip_collision">
-            <origin xyz="-1.8717173055904367e-09 2.8395102015679187e-05 -0.03749999999999909" rpy="3.947037744235681e-16 -0.0 0.0" />
+            <origin xyz="-2.839920353769898e-05 8.17706542477481e-10 -0.0374999999999991" rpy="9.861050790162203e-16 2.814169320963183e-15 1.5707963267948968" />
             <geometry>
                 <mesh filename="package://hexapod_description/meshes/L3_Hip.stl" scale="0.001 0.001 0.001" />
@@ -96,19 +99,19 @@
     <link name="R1_Hip">
         <inertial>
-            <origin xyz="-0.03607404965134453 -0.0008949153164974533 -0.027882386952298888" rpy="0.0 -0.0 0.0" />
+            <origin xyz="0.0008949112149754868 -0.03607404696192064 -0.027882386952298922" rpy="0.0 -0.0 0.0" />
             <mass value="0.6313074615876134" />
-            <inertia ixx="0.0003277483895034669" iyy="0.000395669987103461" izz="0.00025933424464971884" ixy="-7.110381913228742e-06" iyz="-1.8547900647741893e-05" ixz="-1.1372178728115989e-05" />
+            <inertia ixx="0.00039566998710346274" iyy="0.0003277483895034704" izz="0.00025933424464971353" ixy="7.110381913230472e-06" iyz="-1.1372178728115551e-05" ixz="1.8547900647742374e-05" />
         </inertial>
         <visual name="R1_Hip_visual">
-            <origin xyz="-5.436926464597036e-10 -2.8396543466868707e-05 -0.0375000000000004" rpy="3.94703774423568e-16 2.4310372503823276e-15 3.141592653589793" />
+            <origin xyz="2.8392441944902202e-05 2.1457313881256823e-09 -0.03750000000000039" rpy="8.799086709882401e-16 3.731210302817667e-15 -1.5707963267948968" />
             <geometry>
                 <mesh filename="package://hexapod_description/meshes/R1_Hip.stl" scale="0.001 0.001 0.001" />
             </geometry>
             <material name="Red">
-                <color rgba="1.000000 0.000000 0.000000 1.000000"/>
+                <color rgba="1.0 0.0 0.0 1.0"/>
             </material>
         </visual>
         <collision name="R1_Hip_collision">
-            <origin xyz="-5.436926464597036e-10 -2.8396543466868707e-05 -0.0375000000000004" rpy="3.94703774423568e-16 2.4310372503823276e-15 3.141592653589793" />
+            <origin xyz="2.8392441944902202e-05 2.1457313881256823e-09 -0.03750000000000039" rpy="8.799086709882401e-16 3.731210302817667e-15 -1.5707963267948968" />
             <geometry>
                 <mesh filename="package://hexapod_description/meshes/R1_Hip.stl" scale="0.001 0.001 0.001" />
@@ -118,19 +121,19 @@
     <link name="R2_Hip">
         <inertial>
-            <origin xyz="-0.03607404878849106 -0.000894915152145235 -0.027882386952301268" rpy="0.0 -0.0 0.0" />
+            <origin xyz="0.0008949110506231978 -0.03607404609906723 -0.027882386952301347" rpy="0.0 -0.0 0.0" />
             <mass value="0.6313074615876132" />
-            <inertia ixx="0.00032774839016068685" iyy="0.000395669981303616" izz="0.0002593342395016667" ixy="-7.110381836792648e-06" iyz="-1.8547900178346445e-05" ixz="-1.1372180273974968e-05" />
+            <inertia ixx="0.00039566998130361776" iyy="0.00032774839016068706" izz="0.00025933423950166325" ixy="7.1103818367928045e-06" iyz="-1.137218027397532e-05" ixz="1.8547900178346235e-05" />
         </inertial>
         <visual name="R2_Hip_visual">
-            <origin xyz="5.329070518200751e-17 -2.839641866355881e-05 -0.03749999999999999" rpy="3.94703774423568e-16 9.526600354478707e-17 3.141592653589793" />
+            <origin xyz="2.8392317141527902e-05 2.6894238835950547e-09 -0.037499999999999964" rpy="1.042193883590111e-15 2.7334334908028404e-15 -1.5707963267948968" />
             <geometry>
                 <mesh filename="package://hexapod_description/meshes/R2_Hip.stl" scale="0.001 0.001 0.001" />
             </geometry>
             <material name="Red">
-                <color rgba="1.000000 0.000000 0.000000 1.000000"/>
+                <color rgba="1.0 0.0 0.0 1.0"/>
             </material>
         </visual>
         <collision name="R2_Hip_collision">
-            <origin xyz="5.329070518200751e-17 -2.839641866355881e-05 -0.03749999999999999" rpy="3.94703774423568e-16 9.526600354478707e-17 3.141592653589793" />
+            <origin xyz="2.8392317141527902e-05 2.6894238835950547e-09 -0.037499999999999964" rpy="1.042193883590111e-15 2.7334334908028404e-15 -1.5707963267948968" />
             <geometry>
                 <mesh filename="package://hexapod_description/meshes/R2_Hip.stl" scale="0.001 0.001 0.001" />
@@ -140,19 +143,19 @@
     <link name="R3_Hip">
         <inertial>
-            <origin xyz="-0.036074045843427695 -0.0008949187486207677 -0.0278823878445404" rpy="0.0 -0.0 0.0" />
+            <origin xyz="0.0008949146470986769 -0.03607404315400379 -0.0278823878445405" rpy="0.0 -0.0 0.0" />
             <mass value="0.6313073388499953" />
-            <inertia ixx="0.00032774835504940404" iyy="0.0003956699565596661" izz="0.0002593342170091571" ixy="-7.1103939596464246e-06" iyz="-1.854789357175931e-05" ixz="-1.13721841128784e-05" />
+            <inertia ixx="0.000395669956559673" iyy="0.00032774835504940404" izz="0.0002593342170091606" ixy="7.110393959645553e-06" iyz="-1.1372184112877622e-05" ixz="1.854789357176043e-05" />
         </inertial>
         <visual name="R3_Hip_visual">
-            <origin xyz="1.8717173855264947e-09 -2.839773531169598e-05 -0.0374999999999994" rpy="3.947037744235682e-16 -8.475327317661527e-16 3.141592653589793" />
+            <origin xyz="2.8393633789605132e-05 4.561141331294039e-09 -0.037499999999999395" rpy="1.0524000101675127e-15 1.992711098593221e-15 -1.5707963267948968" />
             <geometry>
                 <mesh filename="package://hexapod_description/meshes/R3_Hip.stl" scale="0.001 0.001 0.001" />
             </geometry>
             <material name="Red">
-                <color rgba="1.000000 0.000000 0.000000 1.000000"/>
+                <color rgba="1.0 0.0 0.0 1.0"/>
             </material>
         </visual>
         <collision name="R3_Hip_collision">
-            <origin xyz="1.8717173855264947e-09 -2.839773531169598e-05 -0.0374999999999994" rpy="3.947037744235682e-16 -8.475327317661527e-16 3.141592653589793" />
+            <origin xyz="2.8393633789605132e-05 4.561141331294039e-09 -0.037499999999999395" rpy="1.0524000101675127e-15 1.992711098593221e-15 -1.5707963267948968" />
             <geometry>
                 <mesh filename="package://hexapod_description/meshes/R3_Hip.stl" scale="0.001 0.001 0.001" />
@@ -162,19 +165,19 @@
     <link name="R1_Crus">
         <inertial>
-            <origin xyz="-0.03517075961165982 -4.313120255821091e-06 0.03061202549431937" rpy="0.0 -0.0 0.0" />
-            <mass value="0.19082842966424732" />
-            <inertia ixx="0.00020621482504545917" iyy="0.0003411740602251795" izz="0.0001559819905432797" ixy="9.615429520313057e-10" iyz="2.39260165845511e-08" ixz="3.622540986096274e-08" />
+            <origin xyz="0.030612061044076162 -4.3129226428151316e-06 0.03517075691846999" rpy="0.0 -0.0 0.0" />
+            <mass value="0.19082862947867688" />
+            <inertia ixx="0.0001559819921158473" iyy="0.0003411742204443959" izz="0.00020621498701165527" ixy="2.3924933562503128e-08" iyz="-9.615427496389258e-10" ixz="-3.622538866952052e-08" />
         </inertial>
         <visual name="R1_Crus_visual">
-            <origin xyz="-0.018685768413435184 0.017921808755716372 -0.011675028544473465" rpy="2.9586803559888716e-15 9.464173730837164e-15 -3.141592653589791" />
+            <origin xyz="-0.011675022645995315 0.017921808755716365 0.018685765724011247" rpy="-3.1415926535897913 -1.5707963267948917 0" />
             <geometry>
                 <mesh filename="package://hexapod_description/meshes/R1_Crus.stl" scale="0.001 0.001 0.001" />
             </geometry>
             <material name="Black">
-                <color rgba="0.000000 0.000000 0.000000 1.000000"/>
+                <color rgba="0.0 0.0 0.0 1.0"/>
             </material>
         </visual>
         <collision name="R1_Crus_collision">
-            <origin xyz="-0.018685768413435184 0.017921808755716372 -0.011675028544473465" rpy="2.9586803559888716e-15 9.464173730837164e-15 -3.141592653589791" />
+            <origin xyz="-0.011675022645995315 0.017921808755716365 0.018685765724011247" rpy="-3.1415926535897913 -1.5707963267948917 0" />
             <geometry>
                 <mesh filename="package://hexapod_description/meshes/R1_Crus.stl" scale="0.001 0.001 0.001" />
@@ -184,19 +187,19 @@
     <link name="R2_Crus">
         <inertial>
-            <origin xyz="-0.03482924093203289 4.313120255194925e-06 0.030612025369516436" rpy="0.0 -0.0 0.0" />
-            <mass value="0.19082842966424732" />
-            <inertia ixx="0.00020621482504546004" iyy="0.0003411740602251795" izz="0.00015598199054327883" ixy="9.61542952681756e-10" iyz="-2.3926016585340765e-08" ixz="-3.62254098628518e-08" />
+            <origin xyz="0.030612060919272988 4.31292264206018e-06 0.03482923824637549" rpy="0.0 -0.0 0.0" />
+            <mass value="0.19082862947867688" />
+            <inertia ixx="0.00015598199211584642" iyy="0.0003411742204443959" izz="0.00020621498701165353" ixy="-2.39249335633562e-08" iyz="-9.615427494132688e-10" ixz="3.622538866839477e-08" />
         </inertial>
         <visual name="R2_Crus_visual">
-            <origin xyz="-0.05131423213025757 -0.017921808755717222 -0.01167502866927641" rpy="-3.2267052699708074e-15 2.8845764424670263e-15 2.177306834595132e-16" />
+            <origin xyz="-0.011675022770798318 -0.017921808755717257 0.05131422944083397" rpy="-2.0642981196063126e-15 1.5707963267948917 0" />
             <geometry>
                 <mesh filename="package://hexapod_description/meshes/R2_Crus.stl" scale="0.001 0.001 0.001" />
             </geometry>
             <material name="Black">
-                <color rgba="0.000000 0.000000 0.000000 1.000000"/>
+                <color rgba="0.0 0.0 0.0 1.0"/>
             </material>
         </visual>
         <collision name="R2_Crus_collision">
-            <origin xyz="-0.05131423213025757 -0.017921808755717222 -0.01167502866927641" rpy="-3.2267052699708074e-15 2.8845764424670263e-15 2.177306834595132e-16" />
+            <origin xyz="-0.011675022770798318 -0.017921808755717257 0.05131422944083397" rpy="-2.0642981196063126e-15 1.5707963267948917 0" />
             <geometry>
                 <mesh filename="package://hexapod_description/meshes/R2_Crus.stl" scale="0.001 0.001 0.001" />
@@ -206,19 +209,19 @@
     <link name="R3_Crus">
         <inertial>
-            <origin xyz="-0.034829239060315854 4.313120255874381e-06 0.030612026686164775" rpy="0.0 -0.0 0.0" />
-            <mass value="0.19082842966424732" />
-            <inertia ixx="0.00020621482504546004" iyy="0.00034117406022517865" izz="0.00015598199054327883" ixy="9.615429524649247e-10" iyz="-2.392601658508387e-08" ixz="-3.6225409862044234e-08" />
+            <origin xyz="0.03061206223592098 4.312922642650818e-06 0.034829236374657756" rpy="0.0 -6.357757475712083e-50 0.0" />
+            <mass value="0.19082862947867688" />
+            <inertia ixx="0.0001559819921158473" iyy="0.0003411742204443976" izz="0.0002062149870116531" ixy="-2.392493356315366e-08" iyz="-9.61542749379269e-10" ixz="3.6225388669792216e-08" />
         </inertial>
         <visual name="R3_Crus_visual">
-            <origin xyz="-0.0513142302585405 -0.017921808755716497 -0.011675027352628008" rpy="-2.453621512756187e-15 8.180845673978275e-15 -7.250680518514371e-16" />
+            <origin xyz="-0.011675021454150407 -0.01792180875571667 0.051314227569116466" rpy="-1.821637182365855e-15 1.5707963267948912 0" />
             <geometry>
                 <mesh filename="package://hexapod_description/meshes/R3_Crus.stl" scale="0.001 0.001 0.001" />
             </geometry>
             <material name="Black">
-                <color rgba="0.000000 0.000000 0.000000 1.000000"/>
+                <color rgba="0.0 0.0 0.0 1.0"/>
             </material>
         </visual>
         <collision name="R3_Crus_collision">
-            <origin xyz="-0.0513142302585405 -0.017921808755716497 -0.011675027352628008" rpy="-2.453621512756187e-15 8.180845673978275e-15 -7.250680518514371e-16" />
+            <origin xyz="-0.011675021454150407 -0.01792180875571667 0.051314227569116466" rpy="-1.821637182365855e-15 1.5707963267948912 0" />
             <geometry>
                 <mesh filename="package://hexapod_description/meshes/R3_Crus.stl" scale="0.001 0.001 0.001" />
@@ -228,19 +231,19 @@
     <link name="L1_Crus">
         <inertial>
-            <origin xyz="0.03517075898849346 -4.314155378537521e-06 -0.03061203319839718" rpy="0.0 -0.0 0.0" />
-            <mass value="0.19082842966424732" />
-            <inertia ixx="0.00020621482504546004" iyy="0.00034117406022517865" izz="0.0001559819905432797" ixy="-9.61542952898645e-10" iyz="-2.3926016584556575e-08" ixz="3.622540986258943e-08" />
+            <origin xyz="-0.030612056951197727 -4.313957765593734e-06 -0.0351707616741513" rpy="0.0 -2.285962665308945e-50 0.0" />
+            <mass value="0.19082862947867688" />
+            <inertia ixx="0.0001559819921158473" iyy="0.0003411742204443985" izz="0.00020621498701165484" ixy="-2.392493356261157e-08" iyz="9.615427493389464e-10" ixz="-3.6225388668184415e-08" />
         </inertial>
         <visual name="L1_Crus_visual">
-            <origin xyz="0.018685767790268776 0.017921807720593708 0.011675020840395725" rpy="-3.1415926535897922 -3.556422298105262e-15 -3.77670496181703e-30" />
+            <origin xyz="0.011675026738873715 0.017921807720593638 -0.01868577047969277" rpy="-3.1415926535897927 1.570796326794892 0" />
             <geometry>
                 <mesh filename="package://hexapod_description/meshes/L1_Crus.stl" scale="0.001 0.001 0.001" />
             </geometry>
             <material name="Black">
-                <color rgba="0.000000 0.000000 0.000000 1.000000"/>
+                <color rgba="0.0 0.0 0.0 1.0"/>
             </material>
         </visual>
         <collision name="L1_Crus_collision">
-            <origin xyz="0.018685767790268776 0.017921807720593708 0.011675020840395725" rpy="-3.1415926535897922 -3.556422298105262e-15 -3.77670496181703e-30" />
+            <origin xyz="0.011675026738873715 0.017921807720593638 -0.01868577047969277" rpy="-3.1415926535897927 1.570796326794892 0" />
             <geometry>
                 <mesh filename="package://hexapod_description/meshes/L1_Crus.stl" scale="0.001 0.001 0.001" />
@@ -250,19 +253,19 @@
     <link name="L2_Crus">
         <inertial>
-            <origin xyz="0.0351707590679669 -4.313120255696745e-06 -0.030612025369516665" rpy="0.0 -0.0 0.0" />
-            <mass value="0.19082842966424732" />
-            <inertia ixx="0.00020621482504545988" iyy="0.0003411740602251795" izz="0.00015598199054327883" ixy="-9.615429524649239e-10" iyz="-2.392601658455348e-08" ixz="3.622540986194889e-08" />
+            <origin xyz="-0.030612059122317403 -4.312922642952799e-06 -0.03517076175362483" rpy="0.0 -0.0 0.0" />
+            <mass value="0.19082862947867688" />
+            <inertia ixx="0.00015598199211584556" iyy="0.0003411742204443959" izz="0.00020621498701165267" ixy="-2.392493356254385e-08" iyz="9.615427491882364e-10" ixz="-3.622538866967091e-08" />
         </inertial>
         <visual name="L2_Crus_visual">
-            <origin xyz="0.018685767869742236 0.017921808755716546 0.011675028669276171" rpy="-3.1415926535897922 -8.5685095000437e-15 -9.204085185479184e-30" />
+            <origin xyz="0.01167502456775401 0.017921808755716234 -0.018685770559166155" rpy="-3.1415926535897913 1.5707963267948912 0" />
             <geometry>
                 <mesh filename="package://hexapod_description/meshes/L2_Crus.stl" scale="0.001 0.001 0.001" />
             </geometry>
             <material name="Black">
-                <color rgba="0.000000 0.000000 0.000000 1.000000"/>
+                <color rgba="0.0 0.0 0.0 1.0"/>
             </material>
         </visual>
         <collision name="L2_Crus_collision">
-            <origin xyz="0.018685767869742236 0.017921808755716546 0.011675028669276171" rpy="-3.1415926535897922 -8.5685095000437e-15 -9.204085185479184e-30" />
+            <origin xyz="0.01167502456775401 0.017921808755716234 -0.018685770559166155" rpy="-3.1415926535897913 1.5707963267948912 0" />
             <geometry>
                 <mesh filename="package://hexapod_description/meshes/L2_Crus.stl" scale="0.001 0.001 0.001" />
@@ -272,19 +275,19 @@
     <link name="L3_Crus">
         <inertial>
-            <origin xyz="0.0351707571962495 -4.313120254604285e-06 -0.030612034052867162" rpy="0.0 -0.0 0.0" />
-            <mass value="0.19082842966424732" />
-            <inertia ixx="0.0002062148250454596" iyy="0.0003411740602251804" izz="0.00015598199054328056" ixy="-9.615429526817593e-10" iyz="-2.39260165846797e-08" ixz="3.622540986223205e-08" />
+            <origin xyz="-0.030612057805667874 -4.312922641722672e-06 -0.03517075988190754" rpy="0.0 -0.0 0.0" />
+            <mass value="0.19082862947867688" />
+            <inertia ixx="0.00015598199211584556" iyy="0.0003411742204443976" izz="0.00020621498701165375" ixy="-2.3924933562720035e-08" iyz="9.615427491703478e-10" ixz="-3.622538866997815e-08" />
         </inertial>
         <visual name="L3_Crus_visual">
-            <origin xyz="0.018685765998024823 0.017921808755717642 0.011675019985925648" rpy="-3.1415926535897922 -9.495586488597836e-15 -8.631228484744494e-30" />
+            <origin xyz="0.011675025884403532 0.017921808755717486 -0.018685768687448815" rpy="-3.1415926535897913 1.570796326794891 0" />
             <geometry>
                 <mesh filename="package://hexapod_description/meshes/L3_Crus.stl" scale="0.001 0.001 0.001" />
             </geometry>
             <material name="Black">
-                <color rgba="0.000000 0.000000 0.000000 1.000000"/>
+                <color rgba="0.0 0.0 0.0 1.0"/>
             </material>
         </visual>
         <collision name="L3_Crus_collision">
-            <origin xyz="0.018685765998024823 0.017921808755717642 0.011675019985925648" rpy="-3.1415926535897922 -9.495586488597836e-15 -8.631228484744494e-30" />
+            <origin xyz="0.011675025884403532 0.017921808755717486 -0.018685768687448815" rpy="-3.1415926535897913 1.570796326794891 0" />
             <geometry>
                 <mesh filename="package://hexapod_description/meshes/L3_Crus.stl" scale="0.001 0.001 0.001" />
@@ -294,19 +297,19 @@
     <link name="L1_Foot">
         <inertial>
-            <origin xyz="0.013181239373879201 0.03623956443151984 -0.001257225251094316" rpy="0.0 -0.0 0.0" />
+            <origin xyz="-0.03623955853304191 0.013181242063303174 -0.0012572252510944892" rpy="0.0 -0.0 1.3968124788324058e-47" />
             <mass value="1.073264117385357" />
-            <inertia ixx="0.0013377939900751559" iyy="0.001468280446989316" izz="0.00043109076119057397" ixy="-9.658567712598318e-06" iyz="1.588424012485386e-05" ixz="0.000412185184599299" />
+            <inertia ixx="0.001468280446989316" iyy="0.001337793990075161" izz="0.0004310907611905641" ixy="9.658567712594877e-06" iyz="0.00041218518459930603" ixz="-1.5884240124859086e-05" />
         </inertial>
         <visual name="L1_Foot_visual">
-            <origin xyz="-0.01010000007948257 0.019400003427672525 -0.02056704031521055" rpy="6.610591211137782e-14 9.860761315262522e-32 -7.376125237048963e-48" />
+            <origin xyz="-0.01939999752919466 -0.010099997390058527 -0.020567040315210706" rpy="6.597948698483732e-14 1.2000360668062144e-15 1.5707963267948966" />
             <geometry>
                 <mesh filename="package://hexapod_description/meshes/L1_Foot.stl" scale="0.001 0.001 0.001" />
             </geometry>
             <material name="Red">
-                <color rgba="1.000000 0.000000 0.000000 1.000000"/>
+                <color rgba="1.0 0.0 0.0 1.0"/>
             </material>
         </visual>
         <collision name="L1_Foot_collision">
-            <origin xyz="-0.01010000007948257 0.019400003427672525 -0.02056704031521055" rpy="6.610591211137782e-14 9.860761315262522e-32 -7.376125237048963e-48" />
+            <origin xyz="-0.01939999752919466 -0.010099997390058527 -0.020567040315210706" rpy="6.597948698483732e-14 1.2000360668062144e-15 1.5707963267948966" />
             <geometry>
                 <mesh filename="package://hexapod_description/meshes/L1_Foot.stl" scale="0.001 0.001 0.001" />
@@ -316,19 +319,19 @@
     <link name="L2_Foot">
         <inertial>
-            <origin xyz="0.013181239453366444 0.036239556602639486 -0.0012572242159687886" rpy="0.0 -0.0 0.0" />
+            <origin xyz="-0.036239560704161546 0.013181242142790239 -0.0012572242159690238" rpy="0.0 -0.0 0.0" />
             <mass value="1.0732641173853565" />
-            <inertia ixx="0.001337793990074499" iyy="0.0014682804469887192" izz="0.00043109076119062254" ixy="-9.658567712379743e-06" iyz="1.588424012486442e-05" ixz="0.00041218518460177096" />
+            <inertia ixx="0.0014682804469887262" iyy="0.0013377939900744995" izz="0.0004310907611906335" ixy="9.65856771237967e-06" iyz="0.00041218518460177714" ixz="-1.5884240124871622e-05" />
         </inertial>
         <visual name="L2_Foot_visual">
-            <origin xyz="-0.010100000000000726 0.019399995598791568 -0.02056703928008564" rpy="3.921169725428927e-14 3.697785493220852e-32 -2.766046963891421e-48" />
+            <origin xyz="-0.01939999970031372 -0.01009999731057686 -0.02056703928008582" rpy="3.939058345952069e-14 1.892254372115447e-15 1.5707963267948968" />
             <geometry>
                 <mesh filename="package://hexapod_description/meshes/L2_Foot.stl" scale="0.001 0.001 0.001" />
             </geometry>
             <material name="Red">
-                <color rgba="1.000000 0.000000 0.000000 1.000000"/>
-            </material>
-        </visual>
-        <collision name="L2_Fo_collision">
-            <origin xyz="-0.010100000000000726 0.019399995598791568 -0.02056703928008564" rpy="3.921169725428927e-14 3.697785493220852e-32 -2.766046963891421e-48" />
+                <color rgba="1.0 0.0 0.0 1.0"/>
+            </material>
+        </visual>
+        <collision name="L2_Foot_collision">
+            <origin xyz="-0.01939999970031372 -0.01009999731057686 -0.02056703928008582" rpy="3.939058345952069e-14 1.892254372115447e-15 1.5707963267948968" />
             <geometry>
                 <mesh filename="package://hexapod_description/meshes/L2_Foot.stl" scale="0.001 0.001 0.001" />
@@ -338,19 +341,19 @@
     <link name="L3_Foot">
         <inertial>
-            <origin xyz="0.013181237581652176 0.036239565307096475 -0.0012572242159756275" rpy="0.0 -0.0 0.0" />
+            <origin xyz="-0.036239559408618505 0.013181240271076256 -0.001257224215975925" rpy="0.0 -0.0 1.303429613382641e-47" />
             <mass value="1.0732641173853583" />
-            <inertia ixx="0.0013377939893961677" iyy="0.001468280446984646" izz="0.0004310907605202352" ixy="-9.658567342821192e-06" iyz="1.5884239262163734e-05" ixz="0.0004121851846149002" />
+            <inertia ixx="0.001468280446984653" iyy="0.0013377939893961712" izz="0.0004310907605202392" ixy="9.658567342814282e-06" iyz="0.00041218518461490553" ixz="-1.588423926217156e-05" />
         </inertial>
         <visual name="L3_Foot_visual">
-            <origin xyz="-0.010100001871717198 0.019400004282141385 -0.020567039280084735" rpy="-1.0782612974161142e-15 -2.826793622035183e-44 2.114520685451522e-60" />
+            <origin xyz="-0.0193999983836635 -0.010099999182293082 -0.02056703928008498" rpy="-9.271306678003036e-16 2.3738986459863396e-15 1.5707963267948968" />
             <geometry>
                 <mesh filename="package://hexapod_description/meshes/L3_Foot.stl" scale="0.001 0.001 0.001" />
             </geometry>
             <material name="Red">
-                <color rgba="1.000000 0.000000 0.000000 1.000000"/>
+                <color rgba="1.0 0.0 0.0 1.0"/>
             </material>
         </visual>
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